File: Hardware/Pushbutton v1.0.brd (EAGLE design)
At the start: 24 x 13 mm, 6 parts

Commit message: Add files via upload
Parts:
- moved R1 5.50 mm to (13.7, 9.95)
- moved R2 5.50 mm to (17.5, 9.95), turned to 180 degrees
- moved R3 5.50 mm to (21.3, 9.95), turned to 180 degrees
Routing:
- net PB1: track 11.1 -> 16.7 mm
- net PB3: track 15.6 -> 10.9 mm
- net VCC: track 44.4 -> 42.2 mm
- net PB2: track 10.8 -> 11.9 mm
Other:
- outline, holes or cut-outs redrawn
Changed lines of the file:
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@@
 <wire x1="1" y1="0" x2="23" y2="0" width="0" layer="20"/>
 <wire x1="23" y1="0" x2="24" y2="1" width="0" layer="20"/>
-<wire x1="24" y1="1" x2="24" y2="9" width="0" layer="20"/>
-<wire x1="24" y1="9" x2="23" y2="10" width="0" layer="20"/>
-<wire x1="23" y1="10" x2="20" y2="10" width="0" layer="20"/>
-<wire x1="20" y1="10" x2="19" y2="11" width="0" layer="20"/>
-<wire x1="19" y1="11" x2="19" y2="12" width="0" layer="20"/>
-<wire x1="19" y1="12" x2="18" y2="13" width="0" layer="20"/>
-<wire x1="18" y1="13" x2="6" y2="13" width="0" layer="20"/>
-<wire x1="6" y1="13" x2="5" y2="12" width="0" layer="20"/>
-<wire x1="5" y1="12" x2="5" y2="11" width="0" layer="20"/>
-<wire x1="5" y1="11" x2="4" y2="10" width="0" layer="20"/>
-<wire x1="4" y1="10" x2="1" y2="10" width="0" layer="20"/>
+<wire x1="24" y1="1" x2="24" y2="12" width="0" layer="20"/>
+<wire x1="24" y1="12" x2="23" y2="13" width="0" layer="20"/>
+<wire x1="23" y1="13" x2="12" y2="13" width="0" layer="20"/>
+<wire x1="12" y1="13" x2="11" y2="12" width="0" layer="20"/>
+<wire x1="11" y1="12" x2="11" y2="11" width="0" layer="20"/>
+<wire x1="11" y1="11" x2="10" y2="10" width="0" layer="20"/>
+<wire x1="10" y1="10" x2="1" y2="10" width="0" layer="20"/>
 <wire x1="1" y1="10" x2="0" y2="9" width="0" layer="20"/>
 <wire x1="0" y1="9" x2="0" y2="1" width="0" layer="20"/>
 <wire x1="0" y1="1" x2="1" y2="0" width="0" layer="20"/>
-<text x="18.1" y="9.5" size="0.8" layer="22" font="vector" ratio="15" rot="MR0">GND</text>
-<text x="15.2" y="9.5" size="0.8" layer="22" font="vector" ratio="15" rot="MR0">B3</text>
-<text x="12.65" y="9.5" size="0.8" layer="22" font="vector" ratio="15" rot="MR0">B2</text>
-<text x="10.1" y="9.5" size="0.8" layer="22" font="vector" ratio="15" rot="MR0">B1</text>
-<text x="7.95" y="9.5" size="0.8" layer="22" font="vector" ratio="15" rot="MR0">VCC</text>
+<text x="23.6" y="9.6" size="0.8" layer="22" font="vector" ratio="15" rot="MR0">GND</text>
+<text x="20.7" y="9.6" size="0.8" layer="22" font="vector" ratio="15" rot="MR0">B3</text>
+<text x="18.15" y="9.6" size="0.8" layer="22" font="vector" ratio="15" rot="MR0">B2</text>
+<text x="15.6" y="9.6" size="0.8" layer="22" font="vector" ratio="15" rot="MR0">B1</text>
+<text x="13.45" y="9.6" size="0.8" layer="22" font="vector" ratio="15" rot="MR0">VCC</text>
 <text x="4.65" y="5.5" size="0.8" layer="22" font="vector" ratio="15" rot="MR0">B1</text>
 <text x="12.65" y="5.5" size="0.8" layer="22" font="vector" ratio="15" rot="MR0">B2</text>
@@
 </autorouter>
 <elements>
-<element name="R1" library="TT7" package="RES0402" value="100k" x="8.19" y="9.85" rot="R180"/>
-<element name="R2" library="TT7" package="RES0402" value="100k" x="12" y="9.85"/>
-<element name="R3" library="TT7" package="RES0402" value="100k" x="15.81" y="9.85"/>
+<element name="R1" library="TT7" package="RES0402" value="100k" x="13.69" y="9.95" rot="R180"/>
+<element name="R2" library="TT7" package="RES0402" value="100k" x="17.5" y="9.95" rot="R180"/>
+<element name="R3" library="TT7" package="RES0402" value="100k" x="21.31" y="9.95" rot="R180"/>
 <element name="B1" library="TT7" package="PUSHBUTTON_1" value="PUSHBUTTON_1" x="4" y="5" rot="R90"/>
 <element name="B2" library="TT7" package="PUSHBUTTON_1" value="PUSHBUTTON_1" x="12" y="5" rot="R90"/>
@@
 <vertex x="0" y="0"/>
 </polygon>
-<via x="17.08" y="11.5" extent="1-16" drill="1" diameter="1.6"/>
+<via x="22.58" y="11.7" extent="1-16" drill="1" diameter="1.6"/>
 <contactref element="R1" pad="P$1"/>
 <contactref element="R2" pad="P$1"/>
 <contactref element="R3" pad="P$1"/>
-<via x="8" y="8.5" extent="1-16" drill="0.3" diameter="0.6"/>
-<via x="12" y="8.5" extent="1-16" drill="0.3" diameter="0.6"/>
-<via x="16" y="8.5" extent="1-16" drill="0.3" diameter="0.6"/>
-<via x="20" y="4" extent="1-16" drill="0.3" diameter="0.6"/>
-<via x="4" y="4" extent="1-16" drill="0.3" diameter="0.6"/>
+<via x="8" y="8.6" extent="1-16" drill="0.3" diameter="0.6"/>
+<via x="12" y="8.6" extent="1-16" drill="0.3" diameter="0.6"/>
+<via x="16" y="8.6" extent="1-16" drill="0.3" diameter="0.6"/>
+<via x="20" y="8.6" extent="1-16" drill="0.3" diameter="0.6"/>
+<via x="4" y="8.6" extent="1-16" drill="0.3" diameter="0.6"/>
+<via x="12" y="3.6" extent="1-16" drill="0.3" diameter="0.6"/>
+<via x="20" y="3.6" extent="1-16" drill="0.3" diameter="0.6"/>
+<via x="4" y="3.6" extent="1-16" drill="0.3" diameter="0.6"/>
 </signal>
 <signal name="VCC">
@@
 <contactref element="B3" pad="4"/>
 <contactref element="B3" pad="3"/>
-<via x="6.92" y="11.5" extent="1-16" drill="1" diameter="1.6"/>
+<via x="12.42" y="11.7" extent="1-16" drill="1" diameter="1.6"/>
 <wire x1="1.75" y1="1.75" x2="1.75" y2="8.25" width="0.254" layer="1"/>
 <wire x1="9.75" y1="1.75" x2="9.75" y2="8.25" width="0.254" layer="1"/>
 <wire x1="17.75" y1="1.75" x2="17.75" y2="8.25" width="0.254" layer="1"/>
-<wire x1="6.92" y1="11.5" x2="6.5" y2="11.5" width="0.254" layer="1"/>
-<wire x1="6.5" y1="11.5" x2="4" y2="9" width="0.254" layer="1"/>
-<wire x1="4" y1="9" x2="2.5" y2="9" width="0.254" layer="1"/>
-<wire x1="2.5" y1="9" x2="1.75" y2="8.25" width="0.254" layer="1"/>
-<wire x1="16.6" y1="0.6" x2="9" y2="0.6" width="0.254" layer="1"/>
-<wire x1="9" y1="0.6" x2="2.9" y2="0.6" width="0.254" layer="1"/>
+<wire x1="16.6" y1="0.6" x2="9.75" y2="0.6" width="0.254" layer="1"/>
+<wire x1="9.75" y1="0.6" x2="2.9" y2="0.6" width="0.254" layer="1"/>
 <wire x1="17.75" y1="1.75" x2="16.6" y2="0.6" width="0.254" layer="1"/>
 <wire x1="1.75" y1="1.75" x2="2.9" y2="0.6" width="0.254" layer="1"/>
-<wire x1="9.75" y1="1.75" x2="9.75" y2="1.35" width="0.254" layer="1"/>
-<wire x1="9.75" y1="1.35" x2="9" y2="0.6" width="0.254" layer="1"/>
+<wire x1="9.75" y1="1.75" x2="9.75" y2="0.6" width="0.254" layer="1"/>
+<wire x1="9.75" y1="8.25" x2="9.75" y2="8.75" width="0.254" layer="16"/>
+<wire x1="9.75" y1="8.75" x2="12.42" y2="11.42" width="0.254" layer="16"/>
+<wire x1="12.42" y1="11.42" x2="12.42" y2="11.7" width="0.254" layer="16"/>
 </signal>
 <signal name="PB1">
@@
 <contactref element="R1" pad="P$2"/>
 <contactref element="B1" pad="1"/>
-<via x="9.46" y="11.5" extent="1-16" drill="1" diameter="1.6"/>
+<via x="14.96" y="11.7" extent="1-16" drill="1" diameter="1.6"/>
 <wire x1="6.25" y1="1.75" x2="6.25" y2="8.25" width="0.254" layer="1"/>
 <wire x1="6.25" y1="8.25" x2="6.25" y2="8.41" width="0.254" layer="1"/>
-<wire x1="6.25" y1="8.41" x2="7.69" y2="9.85" width="0.254" layer="1"/>
-<wire x1="7.69" y1="9.85" x2="9.34" y2="11.5" width="0.254" layer="1"/>
-<wire x1="9.34" y1="11.5" x2="9.46" y2="11.5" width="0.254" layer="1"/>
+<wire x1="7.24" y1="9.4" x2="12.64" y2="9.4" width="0.254" layer="1"/>
+<wire x1="6.25" y1="8.41" x2="7.24" y2="9.4" width="0.254" layer="1"/>
+<wire x1="12.64" y1="9.4" x2="13.19" y2="9.95" width="0.254" layer="1"/>
+<wire x1="13.19" y1="9.95" x2="13.21" y2="9.95" width="0.254" layer="1"/>
+<wire x1="13.21" y1="9.95" x2="14.96" y2="11.7" width="0.254" layer="1"/>
 </signal>
 <signal name="PB2">
@@
 <contactref element="R2" pad="P$2"/>
 <contactref element="B2" pad="1"/>
-<via x="12" y="11.5" extent="1-16" drill="1" diameter="1.6"/>
+<via x="17.5" y="11.7" extent="1-16" drill="1" diameter="1.6"/>
 <wire x1="14.25" y1="1.75" x2="14.25" y2="8.25" width="0.254" layer="1"/>
-<wire x1="12" y1="11.5" x2="12.5" y2="11" width="0.254" layer="1"/>
-<wire x1="12.5" y1="11" x2="12.5" y2="9.85" width="0.254" layer="1"/>
-<wire x1="12.5" y1="9.85" x2="12.65" y2="9.85" width="0.254" layer="1"/>
-<wire x1="12.65" y1="9.85" x2="14.25" y2="8.25" width="0.254" layer="1"/>
+<wire x1="14.25" y1="8.25" x2="15.95" y2="9.95" width="0.254" layer="1"/>
+<wire x1="15.95" y1="9.95" x2="17" y2="9.95" width="0.254" layer="1"/>
+<wire x1="17" y1="9.95" x2="17" y2="11.2" width="0.254" layer="1"/>
+<wire x1="17" y1="11.2" x2="17.5" y2="11.7" width="0.254" layer="1"/>
 </signal>
 <signal name="PB3">
@@
 <contactref element="R3" pad="P$2"/>
 <contactref element="B3" pad="1"/>
-<via x="14.54" y="11.5" extent="1-16" drill="1" diameter="1.6"/>
+<via x="20.04" y="11.7" extent="1-16" drill="1" diameter="1.6"/>
 <wire x1="22.25" y1="1.75" x2="22.25" y2="8.25" width="0.254" layer="1"/>
-<wire x1="14.54" y1="11.5" x2="14.66" y2="11.5" width="0.254" layer="1"/>
-<wire x1="14.66" y1="11.5" x2="16.31" y2="9.85" width="0.254" layer="1"/>
-<wire x1="16.31" y1="9.85" x2="19.15" y2="9.85" width="0.254" layer="1"/>
-<wire x1="19.15" y1="9.85" x2="20" y2="9" width="0.254" layer="1"/>
-<wire x1="20" y1="9" x2="21.5" y2="9" width="0.254" layer="1"/>
-<wire x1="21.5" y1="9" x2="22.25" y2="8.25" width="0.254" layer="1"/>
+<wire x1="22.25" y1="8.25" x2="20.81" y2="9.69" width="0.254" layer="1"/>
+<wire x1="20.81" y1="9.69" x2="20.81" y2="9.95" width="0.254" layer="1"/>
+<wire x1="20.81" y1="9.95" x2="20.04" y2="10.72" width="0.254" layer="1"/>
+<wire x1="20.04" y1="10.72" x2="20.04" y2="11.7" width="0.254" layer="1"/>
 </signal>
 </signals>
